File: RP2040-PoE/layouts/default/default.kicad_pcb (KiCad board)
At the start: 2 copper layers, 81.5 x 51.9 mm, 61 parts

Commit message: PoE Improvements
Parts:
- added R17: 270Ω ±1%, UNI_ROYAL_0402WGF2700TCE:R0402, F.Cu at (37.6, 49.2)
- added R18: 270Ω ±1%, UNI_ROYAL_0402WGF2700TCE:R0402, F.Cu at (36.2, 49.2)
- moved C24 11.5 mm to (78.7, 68.4)
- moved R11 7.13 mm to (83.0, 68.5), turned to 90 degrees
- moved C20 6.56 mm to (77.2, 68.4), turned to -90 degrees
- moved R12 5.18 mm to (80.1, 68.4), turned to 90 degrees
- moved R9 3.31 mm to (81.5, 68.4), turned to 90 degrees
- moved C28 0.50 mm to (71.6, 63.2)
- turned C22 to 90 degrees
- turned C27 to 0 degrees
Connections:
- net 3 renamed tx_ct
- net power_3v3-hv renamed 3V3
- net power_5v-hv renamed 5V
- C1 pad 2: lv -> GND
- C10 pad 2: lv -> GND
- C11 pad 2: lv -> GND
- C12 pad 2: lv -> GND
- C13 pad 2: lv -> GND
- C14 pad 2: lv -> GND
- C15 pad 2: input_bypass-power-lv -> lv
- C16 pad 2: input_bypass-power-lv -> lv
- C17 pad 2: lv -> GND
- C18 pad 2: lv -> GND
- C2 pad 2: lv -> GND
- C20 pad 2: lv -> GND
- C21 pad 2: lv -> GND
- C22 pad 2: lv -> GND
- C23 pad 2: lv -> GND
- C24 pad 2: lv -> GND
- C25 pad 2: lv -> GND
- C26 pad 2: lv -> GND
- C27 pad 2: lv -> GND
- C28 pad 2: lv -> GND
- C29 pad 2: lv -> GND
- C3 pad 2: lv -> GND
- C4 pad 2: lv -> GND
- C5 pad 2: lv -> GND
- C6 pad 2: lv -> GND
- C7 pad 2: lv -> GND
- C8 pad 2: lv -> GND
- C9 pad 2: lv -> GND
- D1 pad 2: poe.aux_rectifier-2 -> 2
- R1 pad 2: lv -> GND
- R15 pad 2: lv -> GND
- R16 pad 2: lv -> GND
- R5 pad 2: SDA -> rstn
- R6 pad 2: input_bypass-power-lv -> lv
- RJ1 pad 1: 1 -> phy_tx_n
- RJ1 pad 10: phy_tx_n -> lv
- RJ1 pad 11: phy_rx_p -> activity_led_anode
- RJ1 pad 12: phy_rx_n -> activity_led_cathode
- RJ1 pad 13: 13 -> green_led_anode
- RJ1 pad 14: 14 -> green_led_cathode
- RJ1 pad 2: 2 -> phy_tx_p
- RJ1 pad 4: input_bypass-power-hv -> rx_ct
- RJ1 pad 5: input_bypass-power-hv -> phy_rx_n
- RJ1 pad 6: 6 -> phy_rx_p
- RJ1 pad 7: input_bypass-power-lv -> 7
- RJ1 pad 8: input_bypass-power-lv -> 8
- RJ1 pad 9: phy_tx_p -> input_bypass-power-hv
- RJ1 pad GND1: magjack.jack-GND -> GND
- RJ1 pad GND2: magjack.jack-GND -> GND
- SW1 pad 1: lv -> GND
- SW2 pad 1: lv -> GND
- U1 pad 14: lv -> GND
- U1 pad 16: lv -> GND
- U1 pad 19: lv -> GND
- U1 pad 25: LINKLED -> green_led_cathode
- U1 pad 27: ACTLED -> activity_led_cathode
- U1 pad 29: lv -> GND
- U1 pad 3: lv -> GND
- U1 pad 36: SCL -> eth_int
- U1 pad 37: SDA -> rstn
- U1 pad 48: lv -> GND
- U1 pad 9: lv -> GND
- U2 pad 1: lv -> GND
- U3 pad 1: input_bypass-power-lv -> lv
- U3 pad 10: input_bypass-power-lv -> lv
- U3 pad 7: 7 -> poe.pd-7
- U4 pad 5: lv -> GND
- U5 pad 4: lv -> GND
- U6 pad 12: spi_cs -> cs
- U6 pad 19: lv -> GND
- U6 pad 34: gpio22 -> rstn
- U6 pad 35: gpio23 -> eth_int
- U6 pad 57: lv -> GND
- U6 pad 9: cs -> spi1_cs
- USB1 pad 1: lv -> GND
- USB1 pad 2: lv -> GND
- USB1 pad 3: lv -> GND
- USB1 pad 4: lv -> GND
- USB1 pad A1: lv -> GND
- USB1 pad A12: lv -> GND
- USB1 pad B1: lv -> GND
- USB1 pad B12: lv -> GND
- X1 pad 2: lv -> GND
- X1 pad 4: lv -> GND
Routing:
- net 3V3: track 0.00 -> 200.0 mm, vias 0 -> 6
- net rstn: track 0.00 -> 76.5 mm, vias 0 -> 4
- net eth_int: track 0.00 -> 56.4 mm, vias 0 -> 4
- net MISO: track 0.00 -> 54.9 mm, vias 0 -> 4
- net current_sense_node: track 0.00 -> 48.9 mm
- net cs: track 0.00 -> 47.9 mm, vias 0 -> 4
- net MOSI: track 0.00 -> 46.7 mm, vias 0 -> 4
- net SCLK: track 0.00 -> 45.9 mm, vias 0 -> 2
- net input_bypass-power-hv: track 0.00 -> 41.8 mm
- net lv: track 0.00 -> 40.1 mm, vias 3 -> 2
- net power_1V-hv: track 0.00 -> 38.6 mm, vias 0 -> 2
- net qspi-cs: track 0.00 -> 37.1 mm, vias 0 -> 2
- net 5V: track 0.00 -> 35.9 mm
- net vc_hold-power-hv: track 0.00 -> 35.2 mm
- net clock_load_caps[1]-power-hv: track 0.00 -> 33.6 mm
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- added copper zone on B.Cu, net GND
- added copper zone on F.Cu, net GND
- removed copper zone on B.Cu, net lv
- removed copper zone on F.Cu, net lv
