File: lightbulb/layouts/default/default.kicad_pcb (KiCad board)
At the start: 2 copper layers, 55 x 55 mm, 47 parts

Commit message: First pass of leds
Parts:
- removed ESP32: , Espressif_Systems_ESP32_C3_WROOM_02_N4:BULETM-SMD_ESPRESSIF_ESP32-C3-WROOM-02-N4-4MB
- added U1: , Diodes_Incorporated_AP63301WU_7:TSOT-23-6_L2.9-W1.6-P0.95-LS2.8-BR, F.Cu at (0.00, 0.00)
- C10: value 10µF ±10% -> 100nF ±10%; footprint Samsung_Electro_Mechanics_CL10A106KP8NNNC:C0603 -> YAGEO_CC0603KRX7R9BB104:C0603
- C7: value 1µF ±10% -> 10µF ±10%; footprint Samsung_Electro_Mechanics_CL05A105KA5NQNC:C0402 -> Samsung_Electro_Mechanics_CL10A106KP8NNNC:C0603
- C8: value 10µF ±10% -> 1µF ±10%; footprint Samsung_Electro_Mechanics_CL10A106KP8NNNC:C0603 -> Samsung_Electro_Mechanics_CL05A105KA5NQNC:C0402
- C9: value 100nF ±10% -> 10µF ±10%; footprint YAGEO_CC0603KRX7R9BB104:C0603 -> Samsung_Electro_Mechanics_CL10A106KP8NNNC:C0603
- LED1: footprint HONGLITRONIC_HL_AM_2835D1W_S1_08_HR3_2600K_2800K:LED-SMD_L3.5-W2.8-FD-2835_WHITE -> HONGLITRONIC_HL_AM_2835D1W_S1_08_HR3:LED-SMD_L3.3-W2.8-RD
- LED7: footprint HONGLITRONIC_HL_AM_2835D1W_S1_08_HR3:LED-SMD_L3.3-W2.8-RD -> HONGLITRONIC_HL_AM_2835D1W_S1_08_HR3_2600K_2800K:LED-SMD_L3.5-W2.8-FD-2835_WHITE
- R1: footprint Ever_Ohms_Tech_CR1206FR430P05R:R1206 -> UNI_ROYAL_0603WAF1203T5E:R0603
- R2: footprint UNI_ROYAL_0603WAF1203T5E:R0603 -> UNI_ROYAL_0603WAF3902T5E:R0603
- R3: value 10kΩ ±1% -> (none); footprint UNI_ROYAL_0402WGF1002TCE:R0402 -> Ever_Ohms_Tech_CR1206FR430P05R:R1206
- R5: value 22Ω ±1% -> 10kΩ ±1%; footprint UNI_ROYAL_0402WGF220JTCE:R0402 -> UNI_ROYAL_0402WGF1002TCE:R0402
- R7: value (none) -> 22Ω ±1%; footprint UNI_ROYAL_0603WAF3902T5E:R0603 -> UNI_ROYAL_0402WGF220JTCE:R0402
- U3: footprint Diodes_Incorporated_AP63301WU_7:TSOT-23-6_L2.9-W1.6-P0.95-LS2.8-BR -> Diodes_Incorporated_AL8861WT_7:TSOT-25_L2.9-W1.6-P0.95-LS2.8-BR
- U4: footprint Diodes_Incorporated_AL8861WT_7:TSOT-25_L2.9-W1.6-P0.95-LS2.8-BR -> Espressif_Systems_ESP32_C3_WROOM_02_N4:BULETM-SMD_ESPRESSIF_ESP32-C3-WROOM-02-N4-4MB
- moved C11 322.6 mm to (250.0, -170.0)
- moved R6 292.6 mm to (250.0, -140.0), turned to 0 degrees
- moved C10 289.0 mm to (250.0, -130.0), turned to 0 degrees
- moved L4 271.6 mm to (250.0, -160.0)
- moved C9 268.6 mm to (250.0, -120.0)
- moved R7 267.8 mm to (250.0, -150.0), turned to 0 degrees
- moved R5 264.0 mm to (250.0, -110.0), turned to 0 degrees
- moved C8 263.6 mm to (250.0, -100.0), turned to 0 degrees
- moved R4 237.5 mm to (250.0, -90.0), turned to 0 degrees
- moved C7 231.3 mm to (250.0, -80.0), turned to 0 degrees
- moved L3 208.7 mm to (250.0, -70.0)
- moved L2 203.1 mm to (250.0, -60.0), turned to 0 degrees
- moved C6 200.4 mm to (250.0, -50.0), turned to 0 degrees
- moved C5 189.7 mm to (250.0, -40.0)
- moved C4 180.9 mm to (250.0, -30.0)
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Connections:
- net 1-2 renamed warm_led.channel-1
- net A-10 renamed warm_led-A-3
- net A-11 renamed warm_led-A-4
- net A-2 renamed cool_led-A-1
- net A-4 renamed cool_led-A-3
- net A-9 renamed warm_led-A-2
- C1 pad 2: bst_cap-power-lv -> lv
- C10 pad 1: warm_input_cap-power-hv -> esp32_bypass_cap-power-hv
- C10 pad 2: lv -> input_cap-power-lv
- C11 pad 1: warm_input_cap-power-hv -> input_cap-power-hv
- C11 pad 2: lv -> input_cap-power-lv
- C2 pad 1: warm_input_cap-power-hv -> input_cap-power-hv
- C2 pad 2: lv -> input_cap-power-lv
- C3 pad 1: warm_input_cap-power-hv -> input_cap-power-hv
- C3 pad 2: lv -> input_cap-power-lv
- C4 pad 1: vout_sw-hv -> hv
- C4 pad 2: lv -> input_cap-power-lv
- C5 pad 1: vout_sw-hv -> hv
- C5 pad 2: lv -> input_cap-power-lv
- C6 pad 1: vout_sw-hv -> hv
- C7 pad 1: en_cap-power-hv -> input_cap-power-hv
- C7 pad 2: lv -> input_cap-power-lv
- C8 pad 1: hv -> en_cap-power-hv
- C8 pad 2: lv -> input_cap-power-lv
- C9 pad 1: hv -> esp32_bypass_cap-power-hv
- C9 pad 2: lv -> input_cap-power-lv
- D1 pad 1: warm_input_cap-power-hv -> input_cap-power-hv
- D1 pad 2: A-6 -> A-1
- D2 pad 1: 1-1 -> cool_led.channel-1
- D2 pad 2: lv -> input_cap-power-lv
- D3 pad 2: lv -> input_cap-power-lv
- L1 pad 1: vout_sw-hv -> hv
- L1 pad 2: hv -> esp32_bypass_cap-power-hv
- L2 pad 1: bst_cap-power-lv -> lv
- L2 pad 2: vout_sw-hv -> hv
- L3 pad 2: 1-1 -> cool_led.channel-1
- LED1 pad 1: A-8 -> cool_led-A
- LED1 pad 2: A-7 -> A
- LED10 pad 2: A-7 -> warm_led-A
- LED2 pad 2: A-1 -> cool_led-A
- LED3 pad 1: A-3 -> C
- LED4 pad 1: C -> cool_led-A-2
- LED4 pad 2: A-3 -> A
- LED5 pad 2: A-1 -> cool_led-A-2
- LED6 pad 1: A-5 -> C
- LED7 pad 1: C -> warm_led-A-1
- LED7 pad 2: A-5 -> warm_led-A
- LED8 pad 2: A-8 -> warm_led-A-1
- R1 pad 1: warm_input_cap-power-hv -> hv
- R1 pad 2: A-1 -> fb_cap-power-lv
- R2 pad 1: vout_sw-hv -> fb_cap-power-lv
- R2 pad 2: fb_cap-power-lv -> input_cap-power-lv
- R3 pad 1: hv -> input_cap-power-hv
- R4 pad 1: hv -> esp32_bypass_cap-power-hv
- R4 pad 2: en_cap-power-hv -> esp32-A
- R5 pad 1: A7 -> esp32_bypass_cap-power-hv
- R5 pad 2: 13 -> en_cap-power-hv
- R6 pad 1: A6 -> A7
- R6 pad 2: 14 -> 13
- R7 pad 1: fb_cap-power-lv -> A6
- R7 pad 2: lv -> 14
- R8 pad 1: warm_input_cap-power-hv -> input_cap-power-hv
- R8 pad 2: A-7 -> warm_led-A
- SW1 pad 1: A -> esp32-A
- SW1 pad 2: lv -> input_cap-power-lv
- SW2 pad 2: lv -> input_cap-power-lv
- U2 pad 3: lv -> input_cap-power-lv
- U2 pad 4: warm_input_cap-power-hv -> input_cap-power-hv
- U3 pad 1: fb_cap-power-lv -> cool_led.channel-1
- U3 pad 2: warm_input_cap-power-hv -> input_cap-power-lv
- U3 pad 3: warm_input_cap-power-hv -> 3
- U3 pad 4: lv -> A
- U3 pad 5: bst_cap-power-lv -> input_cap-power-hv
- U4 pad 1: 1-1 -> esp32_bypass_cap-power-hv
- U4 pad 2: lv -> en_cap-power-hv
- U4 pad 4: A-1 -> VSET
- U4 pad 5: warm_input_cap-power-hv -> 5
- U5 pad 2: lv -> input_cap-power-lv
- U5 pad 4: A-7 -> warm_led-A
- U5 pad 5: warm_input_cap-power-hv -> input_cap-power-hv
- USB1 pad 10: lv -> input_cap-power-lv
- USB1 pad 9: lv -> input_cap-power-lv
- USB1 pad B1: lv -> input_cap-power-lv
- USB1 pad B12: lv -> input_cap-power-lv
- USB1 pad B4: A-6 -> A-1
- USB1 pad B9: A-6 -> A-1
Routing:
- net lv: track 190.4 -> 0.00 mm, vias 3 -> 0
- net 23: track 0.00 -> 190.4 mm, vias 0 -> 3
- net warm_input_cap-power-hv: track 134.8 -> 0.00 mm, vias 3 -> 0
- net 31: track 0.00 -> 134.8 mm, vias 0 -> 3
- net hv: track 79.4 -> 0.00 mm, vias 3 -> 0
- net 15: track 0.00 -> 79.4 mm, vias 0 -> 3
- net A-7: track 77.4 -> 0.00 mm, vias 4 -> 0
- net 44: track 0.00 -> 77.4 mm, vias 0 -> 4
- net (no net): track 0.00 -> 70.7 mm
- net warm_led.channel-1: track 67.4 -> 0.00 mm, vias 2 -> 0
- net 33: track 0.00 -> 67.4 mm, vias 0 -> 2
- net 24: track 0.00 -> 50.3 mm, vias 0 -> 2
- net 1-1: track 50.3 -> 0.00 mm, vias 2 -> 0
- net vout_sw-hv: track 46.4 -> 0.00 mm
- net 43: track 0.00 -> 46.4 mm
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